File: 01 Hardware/13 lighting/01 Hardware/01 sheet/Lighting.sch (EAGLE design)
At the start: 58 parts, among them IC1 AD822R, IC2 AD822R, J2 614105150721, J3 690367290476, J4 690367291276, U10 Grün, U11 Rot, U7 W1, U8 W2

Commit message: new Lighting PCB
Parts:
- removed J2: 614105150721, Eagle_WR-USB (rev24c):614105150721
- added J1: 614105150621, Eagle_WR-USB (rev25c):614105150621
- GRUEN: value LED_PLATINE -> GRUEN
- ROT: value LED_PLATINE -> ROT
- U$1: value RP2350_STAMPTHT -> RP2350_STAMPSMD; device rp2xxx_stamp:RP2350_STAMPTHT -> rp2xxx_stamp:RP2350_STAMPSMD
- W11: value LED_PLATINE -> W11
- W12: value LED_PLATINE -> W12
- W13: value LED_PLATINE -> W13
- W21: value LED_PLATINE -> W21
- W22: value LED_PLATINE -> W22
- W23: value LED_PLATINE -> W23
Connections:
- net +5V: now also D5.C; no longer D5.A
- net D+@1: now also J1.D+; no longer J2.D+
- net D-@1: now also J1.D-; no longer J2.D-
- net GND: now also GRUEN.5, J1.GND, J1.SHIELD, ROT.5, W11.5, W12.5, W13.5, W21.5, W22.5, W23.5; no longer J2.GND
- net PD_W1: no longer W12.4, W13.4
- net PD_W2: no longer W21.4, W22.4
- net VBUS: now also D5.A, J1.VBUS; no longer D5.C, J2.VBUS
